Commit message: Update depthai_macro.urdf.xacro

File: depthai_descriptions/urdf/include/depthai_macro.urdf.xacro (robot description, xacro)
@@ -19,4 +19,13 @@
       <xacro:property name="imu_p" value="1.5708" />
       <xacro:property name="imu_y" value="0" />
+    </xacro:if>
+    <xacro:if value="${model == 'OAK-D-PRO'}">
+      <xacro:property name="has_imu" value="true" />
+      <xacro:property name="imu_offset_x" value="-0.008" />
+      <xacro:property name="imu_offset_y" value="-0.037945" />
+      <xacro:property name="imu_offset_z" value="-0.00079" />
+      <xacro:property name="imu_r" value="${M_PI}" />
+      <xacro:property name="imu_p" value="${M_PI/2.0}" />
+      <xacro:property name="imu_y" value="0.0" />
     </xacro:if>
     <!-- base_link of the sensor-->
